File: dvi-sock.kicad_sch (KiCad schematic)
At the start: 12 parts, among them J1 Conn_01x05, J2 Conn_01x05, J3 Conn_01x03, J4 NOT_HDMI_A

Commit message: Tweak clock lane grounding, add optional 5V header
Parts:
- added J5: 2.54mm_2p_nofit, dvi-sock:PinHeader_1x02_P2.54mm_Vertical_nosilk, symbol Connector_Generic:Conn_01x02
Connections:
- net GND: now also J5.2 (Pin_2)
- net +5V: now reaches J4.18 (+5V)
- net +5V: now also J5.1 (Pin_1)
- no-connect marks 8 -> 7
Other:
- note added: "Optional 5V Header (no-fit)"
- note added: "Socket which I can't say the name of"
- note added: "Surface mount footprint for the non-USB end of a RPi Pico"
- note added: "You're supposed to drive the 5V line before outputting video (it's part of a nominal startup state machine in the DVI spec, not just for supplying the DDC + EDID). However most monitors don't seem to care, and the VBUS pin is at the far end of Pico, so this board just hooks up the grounds and the TMDS lanes, not the +5V. If you have trouble you can fit this header and supply 5V to the Sink throug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"
- moved on the sheet: J1, J2, J3, J4, R1, R2, R3, R4, R5, R6, R7, R8

Commit message: Update name/date on schematic
Other:
- company: (none) -> Luke Wren
Changed lines of the file:
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@@
   (title_block
     (title "Pico DVI Sock (or Shim, or something, idk what to call it)")
-    (date "2021-02-01")
+    (date "2021-02-02")
     (rev "A")
+    (company "Luke Wren")
     (comment 1 "and stick the board into a breadboard. Micro-USB one end, video the other end.")
     (comment 2 "low-profile on the bottom, so you can fit headers to the remaining Pico I/O pins")
